File: backbone.kicad_pcb (KiCad board)
At the start: 2 copper layers, 20 parts, among them J10 Conn_01x04, J11 Conn_01x04, J12 DEL, J2 Servo 1, J3 Servo 2, J4 Pont en H 1, J5 Pont en H 1, J6 SPI, J7 I2C, J8 Conn_01x04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

Commit message: wip
Parts:
- removed J10, J9: Conn_01x04, Connector_PinHeader_2.54mm:PinHeader_1x04_P2.54mm_Vertical
- removed J6: SPI, Connector_PinHeader_2.54mm:PinHeader_1x06_P2.54mm_Vertical
- removed JP5: Jumper_2_Bridged, Connector_PinHeader_2.54mm:PinHeader_1x02_P2.54mm_Vertical
- added C1: 1u, Capacitor_SMD:C_0805_2012Metric_Pad1.18x1.45mm_HandSolder, F.Cu at (176.5, 78.0)
- added C2: 1u, Capacitor_SMD:C_0805_2012Metric_Pad1.18x1.45mm_HandSolder, F.Cu at (100.3, 119.4)
- added C3: 1u, Capacitor_SMD:C_0805_2012Metric_Pad1.18x1.45mm_HandSolder, F.Cu at (113.0, 119.4)
- added C4: 1u, Capacitor_SMD:C_0805_2012Metric_Pad1.18x1.45mm_HandSolder, F.Cu at (162.3, 118.1)
- added C5: 1u, Capacitor_SMD:C_0805_2012Metric_Pad1.18x1.45mm_HandSolder, F.Cu at (136.9, 116.8)
- added D1: SM4001, Diode_SMD:D_MELF, F.Cu at (116.5, 105.3)
- added D2: LED, LED_SMD:LED_0805_2012Metric_Pad1.15x1.40mm_HandSolder, F.Cu at (98.8, 59.7)
- added D3: LED, LED_SMD:LED_0805_2012Metric_Pad1.15x1.40mm_HandSolder, F.Cu at (98.8, 63.5)
- added D4: LED, LED_SMD:LED_0805_2012Metric_Pad1.15x1.40mm_HandSolder, F.Cu at (98.8, 67.3)
- added D5: LED, LED_SMD:LED_0805_2012Metric_Pad1.15x1.40mm_HandSolder, F.Cu at (98.8, 71.1)
- added FID1: Fiducial, Fiducial:Fiducial_1.5mm_Mask4.5mm, F.Cu at (106.0, 50.0)
- added FID2: Fiducial, Fiducial:Fiducial_1.5mm_Mask4.5mm, F.Cu at (180.0, 124.0)
- added H1: MountingHole_Pad, MountingHole:MountingHole_3.2mm_M3_DIN965_Pad, F.Cu at (100.0, 50.0)
- added H2: MountingHole_Pad, MountingHole:MountingHole_3.2mm_M3_DIN965_Pad, F.Cu at (180.0, 50.0)
- added H3: MountingHole_Pad, MountingHole:MountingHole_3.2mm_M3_DIN965_Pad, F.Cu at (180.0, 130.0)
- added H4: MountingHole_Pad, MountingHole:MountingHole_3.2mm_M3_DIN965_Pad, F.Cu at (100.0, 130.0)
- added J1: Conn_01x05, Library:Carte_alimentation, F.Cu at (117.9, 57.9)
- added R3: 330, Resistor_SMD:R_0805_2012Metric_Pad1.20x1.40mm_HandSolder, F.Cu at (103.9, 59.7)
- added R4: 330, Resistor_SMD:R_0805_2012Metric_Pad1.20x1.40mm_HandSolder, F.Cu at (103.9, 63.5)
- added R5: 330, Resistor_SMD:R_0805_2012Metric_Pad1.20x1.40mm_HandSolder, F.Cu at (103.9, 67.3)
- added R6: 330, Resistor_SMD:R_0805_2012Metric_Pad1.20x1.40mm_HandSolder, F.Cu at (103.9, 71.1)
- added R7: 0, Resistor_SMD:R_0805_2012Metric_Pad1.20x1.40mm_HandSolder, F.Cu at (167.6, 78.2)
- added U2: SN74LVC2G14DBV, Package_TO_SOT_SMD:SOT-23-6, F.Cu at (160.9, 56.1)
- J11: value Conn_01x04 -> UART
- J4: value Pont en H 1 -> Pont en H
- J5: value Pont en H 1 -> Conn_01x07; footprint Connector_PinHeader_2.54mm:PinHeader_1x06_P2.54mm_Vertical -> Connector_PinHeader_2.54mm:PinHeader_1x07_P2.54mm_Vertical
- J8: value Conn_01x04 -> Capteur Distance
- R1, R2: value R -> 5.1k; footprint Resistor_SMD:R_0805_2012Metric -> Resistor_SMD:R_0805_2012Metric_Pad1.20x1.40mm_HandSolder
- moved J5 47.3 mm to (172.7, 106.1), turned to 0 degrees
- moved R2 24.0 mm to (168.9, 90.9), turned to -90 degrees
- moved J2 23.4 mm to (104.1, 121.9)
- moved J8 22.9 mm to (157.5, 121.9)
- moved J7 22.7 mm to (172.7, 89.6)
- moved R1 21.4 mm to (176.5, 90.9), turned to -90 degrees
- moved JP1 20.4 mm to (111.8, 59.7), turned to -90 degrees
- moved JP6 16.5 mm to (128.3, 121.9), turned to 180 degrees
- moved J4 16.4 mm to (154.6, 51.1)
- moved U1 15.9 mm to (152.1, 83.8)
- moved J11 14.9 mm to (133.3, 121.9)
- moved J3 13.7 mm to (109.2, 121.9)
- moved JP2 11.6 mm to (111.8, 63.5), turned to -90 degrees
- moved J12 10.2 mm to (172.7, 76.2)
- moved JP4 6.46 mm to (111.8, 71.1), turned to -90 degrees
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Connections:
- net /CH-D_EN renamed /CS2
- net /CH-D_IN4 renamed /CS1
- J12 pad 2: /DOUT -> Net-(J12-Pin_2)
- J5 pad 1: /CH-C_EN -> 3V3
- J5 pad 2: /CH-C_IN1 -> /SCK
- J5 pad 3: /CH-C_IN2 -> /MOSI
- J5 pad 4: /CH-D_IN3 -> /MISO
- U1 pad 1: unconnected-(U1-D1-Pad1) -> /PWM_2
- U1 pad 12: unconnected-(U1-D9-Pad12) -> /PWM_1
- U1 pad 15: unconnected-(U1-D12-Pad15) -> /SDA
- U1 pad 2: unconnected-(U1-D0-Pad2) -> /RX
- U1 pad 21: unconnected-(U1-A6-Pad21) -> /SCL
- U1 pad 22: unconnected-(U1-A5-Pad22) -> /MISO
- U1 pad 26: unconnected-(U1-A1-Pad26) -> /SCK
- U1 pad 5: unconnected-(U1-D2-Pad5) -> /MOSI
- U1 pad 8: unconnected-(U1-D5-Pad8) -> /TX
Other:
- board outline added: 90 x 90 mm
- board text added: "Carte d'alimentation"
- board text added: "Distance"
- board text added: "I2C"
- board text added: "LED"
- board text added: "Moteurs DC"
- board text added: "P/N : 0000 S/N : 0001"
- board text added: "SPI"
- board text added: "Servo Moteurs"
- board text added: "UART"
