File: backbone.kicad_sch (KiCad schematic)
At the start: 30 parts, among them J1 Conn_01x05, J10 Conn_01x04, J11 Conn_01x04, J12 DEL, J2 Servo 1, J3 Servo 2, J4 Pont en H 1, J5 Pont en H 1, J6 SPI, J7 I2C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

Commit message: wip
Parts:
- removed D1: D, symbol Device:D
- removed J10, J9: Conn_01x04, Connector_PinHeader_2.54mm:PinHeader_1x04_P2.54mm_Vertical, symbol Connector_Generic:Conn_01x04
- removed J5: Pont en H 1, Connector_PinHeader_2.54mm:PinHeader_1x06_P2.54mm_Vertical, symbol Connector_Generic:Conn_01x06
- removed J6: SPI, Connector_PinHeader_2.54mm:PinHeader_1x06_P2.54mm_Vertical, symbol Connector_Generic:Conn_01x06
- removed JP5: Jumper_2_Bridged, Connector_PinHeader_2.54mm:PinHeader_1x02_P2.54mm_Vertical, symbol Jumper:Jumper_2_Bridged
- added C1, C2, C3, C4, C5: 1u, Capacitor_SMD:C_0805_2012Metric_Pad1.18x1.45mm_HandSolder, symbol Device:C
- added D1: SM4001, Diode_SMD:D_MELF, symbol Diode:SM4001
- added FID1, FID2: Fiducial, Fiducial:Fiducial_1.5mm_Mask4.5mm, symbol Mechanical:Fiducial
- added H1, H2, H3, H4: MountingHole_Pad, MountingHole:MountingHole_3.2mm_M3_DIN965_Pad, symbol Mechanical:MountingHole_Pad
- added J5: Conn_01x07, Connector_PinHeader_2.54mm:PinHeader_1x07_P2.54mm_Vertical, symbol Connector_Generic:Conn_01x07
- added R7: 0, Resistor_SMD:R_0805_2012Metric_Pad1.20x1.40mm_HandSolder, symbol Device:R
- added U2: SN74LVC2G14DBV, Package_TO_SOT_SMD:SOT-23-6, symbol 74xGxx:SN74LVC2G14DBV
- D2, D3, D4, D5: footprint (none) -> LED_SMD:LED_0805_2012Metric_Pad1.15x1.40mm_HandSolder
- J1: footprint (none) -> Library:Carte_alimentation
- J11: value Conn_01x04 -> UART
- J4: value Pont en H 1 -> Pont en H
- J8: value Conn_01x04 -> Capteur Distance
- R1, R2, R3, R4, R5, R6: footprint Resistor_SMD:R_0805_2012Metric -> Resistor_SMD:R_0805_2012Metric_Pad1.20x1.40mm_HandSolder
Connections:
- net 3V3: now also C1.1, C4.1, J5.1 (Pin_1), U2.5 (V_{CC})
- net 7.4V: now also C2.1, C3.1, D1.2 (A)
- net CH-A_IN1: now also U2.1 (1A)
- net CH-A_IN2: now also U2.6 (1Y)
- net CH-B_IN3: now also U2.3 (2A)
- net CH-B_IN4: now also U2.4 (2Y)
- net DOUT: now also R7.1; no longer J12.2 (Pin_2)
- net GND: now also J1.5 (Pin_5), C1.2, C2.2, C3.2, C4.2, C5.2, H1.1, H2.1, H3.1, H4.1, J5.7 (Pin_7), U2.2 (GND)
- net MISO: now also U1.22 (A5), J5.4 (Pin_4)
- net MOSI: now also U1.5 (D2), J5.3 (Pin_3)
- net PWM_1: now also U1.12 (D9)
- net PWM_2: now also U1.1 (D1)
- net RX: now also U1.2 (D0)
- net SCK: now also U1.26 (A1), J5.2 (Pin_2)
- net SCL: now also U1.21 (A6)
- net SDA: now also U1.15 (D12)
- net TX: now also U1.8 (D5)
- net at U1.16 (VIN): now also D1.1 (K)
- net at J11.1 (Pin_1), JP6.2 (C): now also C5.1
- new net: J12.2 (Pin_2), R7.2
- new net CS1: J5.5 (Pin_5)
- new net CS2: J5.6 (Pin_6)
Other:
- moved on the sheet: D2, D3, D4, D5, J1, J11, J12, J2, J3, J4, J7, J8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
